File: led-board/led-board.kicad_sch (KiCad schematic)
At the start: 2 parts

Commit message: layout: place and route LED circuit
Parts:
- D1: footprint (none) -> LED_THT:LED_D5.0mm
- R1: footprint (none) -> Resistor_THT:R_Axial_DIN0309_L9.0mm_D3.2mm_P12.70mm_Horizontal
Changed lines of the file:
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@@
 			)
 		)
-		(property "Footprint" ""
+		(property "Footprint" "Resistor_THT:R_Axial_DIN0309_L9.0mm_D3.2mm_P12.70mm_Horizontal"
 			(at 137.16 84.328 90)
 			(hide yes)
@@
 			)
 		)
-		(property "Footprint" ""
+		(property "Footprint" "LED_THT:LED_D5.0mm"
 			(at 128.27 82.55 0)
 			(hide yes)
